File: hardware/cpu_board/untitled.sch (EAGLE design)
At the start: 70 parts, among them IC1 MAX232ECWE, IC2 MAX232ECWE, IC3 AM29F040J, IC4 74HCT138D, IC5 LM2596S, J2 POWER_JACKSLT, U1 AS6C4008-55SIN

Commit message: PCB update
Connections:
- net !BUSACK: now also U$4.!BUSACK
- net !BUSREQ: now also U$4.!BUSREQ
- net !INT: now also U$4.!INT0
- net !IRQ1: now also U$4.!INT1
- net !IRQ2: now also U$4.!INT2
- net !NMI: now also U$4.!NMI
- net !RD: now also U$4.!RD
- net !RST: now also U$4.!RESET
- net !WAIT: now also U$4.!WAIT
- net !WR: now also U$4.!WR
- net 5V: now also U$4.VCC@1
- net A0: now also U$4.A0
- net A1: now also U$4.A1
- net A10: now also U$4.A10
- net A11: now also U$4.A11
- net A12: now also U$4.A12
- net A13: now also U$4.A13
- net A14: now also U$4.A14
- net A15: now also U$4.A15
- net A16: now also U$4.A16
- net A17: now also U$4.A17
- net A18: now also U$4.A18/TOUT
- net A2: now also U$4.A2
- net A3: now also U$4.A3
- net A4: now also U$4.A4
- net A5: now also U$4.A5
- net A6: now also U$4.A6
- net A7: now also U$4.A7
- net A8: now also U$4.A8
- net A9: now also U$4.A9
- net CLK: now also U$4.CLK
- net CTS1: now also U$4.!CTS0
- net CTS2: now also U$4.RXS/!CTS1
- net D0: now also U$4.D0
- net D1: now also U$4.D1
- net D2: now also U$4.D2
- net D3: now also U$4.D3
- net D4: now also U$4.D4
- net D5: now also U$4.D5
- net D6: now also U$4.D6
- net D7: now also U$4.D7
- net GND: now also U$4.VSS@1, U$4.VSS@2, U$4.VSS@3, U$4.VSS@4
- net RTS1: now also U$4.!RTS0
- net RXD1: now also U$4.RXA0
- net RXD2: now also U$4.RXA1
- net ST: now also U$4.ST
- net TXD1: now also U$4.TXA0
- net TXD2: now also U$4.TXA1
Other:
- moved on the sheet: R14

Commit message: PCB updated
Parts:
- removed U$3: ASE, crystal:ASE
- added C16, C32: (no value), rcl:C-EUC0603
- added Y1: CRYSTAL-GROUNDEDSMD-5X3.2, SparkFun-Clocks:CRYSTAL-GROUNDEDSMD-5X3.2
- R4, R6: device rcl:R-EU_R0603 -> rcl:R-EU_R0402
Connections:
- removed net OSC_IN: U$3.OUT
- new net EXTAL: C16.1, U$4.EXTAL, Y1.1
- new net XTAL: C32.1, U$4.XTAL, Y1.2
- net 5V: no longer U$3.VDD
- net GND: now also C16.2, C32.2, Y1.3; no longer U$3.GND
Changed lines of the file:
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@@
 <part name="GND10" library="supply1" deviceset="GND" device=""/>
 <part name="C17" library="rcl" deviceset="C-EU" device="C0603"/>
-<part name="R4" library="rcl" deviceset="R-EU_" device="R0603"/>
+<part name="R4" library="rcl" deviceset="R-EU_" device="R0402"/>
 <part name="R5" library="rcl" deviceset="R-EU_" device="R1206"/>
 <part name="JP2" library="pinhead" deviceset="PINHD-2X4" device=""/>
@@
 <part name="RN1" library="resistor-sil" deviceset="G04R" device=""/>
 <part name="R3" library="rcl" deviceset="R-EU_" device="R0402"/>
-<part name="R6" library="rcl" deviceset="R-EU_" device="R0603"/>
+<part name="R6" library="rcl" deviceset="R-EU_" device="R0402"/>
 <part name="U$2" library="mw" deviceset="TL7705" device=""/>
 <part name="GND11" library="supply1" deviceset="GND" device=""/>
@@
 <part name="JP10" library="pinhead" deviceset="PINHD-1X8" device=""/>
 <part name="JP11" library="pinhead" deviceset="PINHD-1X18" device=""/>
-<part name="U$3" library="crystal" deviceset="ASE" device=""/>
-<part name="GND74" library="supply1" deviceset="GND" device=""/>
 <part name="C15" library="rcl" deviceset="C-EU" device="C0603"/>
 <part name="U$4" library="mw" deviceset="HD64180" device=""/>
 <part name="GND9" library="supply1" deviceset="GND" device=""/>
+<part name="C16" library="rcl" deviceset="C-EU" device="C0603"/>
+<part name="C32" library="rcl" deviceset="C-EU" device="C0603"/>
+<part name="GND17" library="supply1" deviceset="GND" device=""/>
+<part name="GND35" library="supply1" deviceset="GND" device=""/>
+<part name="Y1" library="SparkFun-Clocks" deviceset="CRYSTAL-GROUNDED" device="SMD-5X3.2"/>
+<part name="GND22" library="supply1" deviceset="GND" device=""/>
 </parts>
 <sheets>
@@
 <instance part="JP10" gate="A" x="464.82" y="177.8" rot="MR180"/>
 <instance part="JP11" gate="A" x="464.82" y="129.54" rot="MR180"/>
-<instance part="U$3" gate="G$1" x="-33.02" y="116.84"/>
-<instance part="GND74" gate="1" x="-48.26" y="104.14"/>
 <instance part="C15" gate="G$1" x="-119.38" y="190.5"/>
 <instance part="U$4" gate="G$1" x="86.36" y="276.86"/>
 <instance part="GND9" gate="1" x="45.72" y="223.52"/>
+<instance part="C16" gate="G$1" x="-33.02" y="149.86"/>
+<instance part="C32" gate="G$1" x="-40.64" y="149.86"/>
+<instance part="GND17" gate="1" x="-33.02" y="132.08"/>
+<instance part="GND35" gate="1" x="-40.64" y="132.08"/>
+<instance part="Y1" gate="G$1" x="-33.02" y="160.02" rot="R90"/>
+<instance part="GND22" gate="1" x="-25.4" y="132.08"/>
 </instances>
 <busses>
@@
 </segment>
 <segment>
-<pinref part="U$3" gate="G$1" pin="GND"/>
-<pinref part="GND74" gate="1" pin="GND"/>
-<wire x1="-45.72" y1="111.76" x2="-48.26" y2="111.76" width="0.1524" layer="91"/>
-<wire x1="-48.26" y1="111.76" x2="-48.26" y2="106.68" width="0.1524" layer="91"/>
-</segment>
-<segment>
 <pinref part="U$4" gate="G$1" pin="VSS@1"/>
 <pinref part="GND9" gate="1" pin="GND"/>
@@
 <wire x1="88.9" y1="320.04" x2="88.9" y2="317.5" width="0.1524" layer="91"/>
 <junction x="86.36" y="320.04"/>
+</segment>
+<segment>
+<pinref part="C16" gate="G$1" pin="2"/>
+<pinref part="GND17" gate="1" pin="GND"/>
+<wire x1="-33.02" y1="134.62" x2="-33.02" y2="144.78" width="0.1524" layer="91"/>
+</segment>
+<segment>
+<pinref part="C32" gate="G$1" pin="2"/>
+<pinref part="GND35" gate="1" pin="GND"/>
+<wire x1="-40.64" y1="134.62" x2="-40.64" y2="144.78" width="0.1524" layer="91"/>
+</segment>
+<segment>
+<pinref part="Y1" gate="G$1" pin="3"/>
+<pinref part="GND22" gate="1" pin="GND"/>
+<wire x1="-27.94" y1="160.02" x2="-25.4" y2="160.02" width="0.1524" layer="91"/>
+<wire x1="-25.4" y1="160.02" x2="-25.4" y2="134.62" width="0.1524" layer="91"/>
 </segment>
 </net>
@@
 </segment>
 <segment>
-<pinref part="U$3" gate="G$1" pin="VDD"/>
-<wire x1="-45.72" y1="121.92" x2="-48.26" y2="121.92" width="0.1524" layer="91"/>
-<wire x1="-48.26" y1="121.92" x2="-48.26" y2="129.54" width="0.1524" layer="91"/>
-<label x="-48.26" y="129.54" size="1.4224" layer="95" rot="R90" xref="yes"/>
-</segment>
-<segment>
 <pinref part="U$4" gate="G$1" pin="VCC@1"/>
 <wire x1="86.36" y1="233.68" x2="86.36" y2="226.06" width="0.1524" layer="91"/>
@@
 <label x="22.86" y="78.74" size="1.4224" layer="95" rot="R180" xref="yes"/>
 </segment>
-<segment>
-<pinref part="U$3" gate="G$1" pin="OUT"/>
-<wire x1="-20.32" y1="116.84" x2="-12.7" y2="116.84" width="0.1524" layer="91"/>
-<label x="-12.7" y="116.84" size="1.4224" layer="95" rot="MR180" xref="yes"/>
-</segment>
 </net>
 <net name="N$25" class="0">
@@
 </segment>
 </net>
+<net name="XTAL" class="0">
+<segment>
+<pinref part="U$4" gate="G$1" pin="XTAL"/>
+<wire x1="83.82" y1="317.5" x2="83.82" y2="325.12" width="0.1524" layer="91"/>
+<label x="83.82" y="325.12" size="1.4224" layer="95" rot="R90" xref="yes"/>
+</segment>
+<segment>
+<wire x1="-20.32" y1="165.1" x2="-33.02" y2="165.1" width="0.1524" layer="91"/>
+<wire x1="-33.02" y1="165.1" x2="-33.02" y2="162.56" width="0.1524" layer="91"/>
+<pinref part="C32" gate="G$1" pin="1"/>
+<wire x1="-33.02" y1="165.1" x2="-40.64" y2="165.1" width="0.1524" layer="91"/>
+<wire x1="-40.64" y1="165.1" x2="-40.64" y2="152.4" width="0.1524" layer="91"/>
+<junction x="-33.02" y="165.1"/>
+<pinref part="Y1" gate="G$1" pin="2"/>
+<wire x1="-20.32" y1="165.1" x2="-12.7" y2="165.1" width="0.1524" layer="91"/>
+<label x="-12.7" y="165.1" size="1.4224" layer="95" xref="yes"/>
+</segment>
+</net>
+<net name="EXTAL" class="0">
+<segment>
+<pinref part="U$4" gate="G$1" pin="EXTAL"/>
+<wire x1="78.74" y1="317.5" x2="78.74" y2="325.12" width="0.1524" layer="91"/>
+<label x="78.74" y="325.12" size="1.4224" layer="95" rot="R90" xref="yes"/>
+</segment>
+<segment>
+<wire x1="-12.7" y1="154.94" x2="-33.02" y2="154.94" width="0.1524" layer="91"/>
+<wire x1="-33.02" y1="154.94" x2="-33.02" y2="157.48" width="0.1524" layer="91"/>
+<pinref part="C16" gate="G$1" pin="1"/>
+<wire x1="-33.02" y1="154.94" x2="-33.02" y2="152.4" width="0.1524" layer="91"/>
+<junction x="-33.02" y="154.94"/>
+<pinref part="Y1" gate="G$1" pin="1"/>
+<label x="-12.7" y="154.94" size="1.4224" layer="95" xref="yes"/>
+</segment>
+</net>

Commit message: PCB updated
Parts:
- removed C16, C32: (no value), rcl:C-EUC0603
- removed Y1: CRYSTAL-GROUNDEDSMD-5X3.2, SparkFun-Clocks:CRYSTAL-GROUNDEDSMD-5X3.2
- added R11: (no value), rcl:R-EU_R0603
- added U$3: ASE, crystal:ASE
- R15: device rcl:R-EU_R0402 -> rcl:R-EU_R0603
Connections:
- new net N$26: IC4A.G1, R11.1
- net !IORQ: now also U$4.!IOE
- net !M1: no longer IC4A.G1
- net 5V: now also R11.2, U$3.VDD
- net EXTAL: now also U$3.OUT; no longer C16.1, Y1.1
- net GND: now also U$3.GND; no longer C16.2, C32.2, Y1.3
- net N$25: now also U$4.!DREQ1
- net XTAL: no longer C32.1, Y1.2
Other:
- moved on the sheet: R15
Changed lines of the file:
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@@
 <part name="GND26" library="supply1" deviceset="GND" device=""/>
 <part name="R14" library="rcl" deviceset="R-EU_" device="0204/5"/>
-<part name="R15" library="rcl" deviceset="R-EU_" device="R0402"/>
+<part name="R15" library="rcl" deviceset="R-EU_" device="R0603"/>
 <part name="C29" library="rcl" deviceset="C-EU" device="C0603"/>
 <part name="C30" library="rcl" deviceset="CPOL-EU" device="SMCB"/>
@@
 <part name="U$4" library="mw" deviceset="HD64180" device=""/>
 <part name="GND9" library="supply1" deviceset="GND" device=""/>
-<part name="C16" library="rcl" deviceset="C-EU" device="C0603"/>
-<part name="C32" library="rcl" deviceset="C-EU" device="C0603"/>
-<part name="GND17" library="supply1" deviceset="GND" device=""/>
-<part name="GND35" library="supply1" deviceset="GND" device=""/>
-<part name="Y1" library="SparkFun-Clocks" deviceset="CRYSTAL-GROUNDED" device="SMD-5X3.2"/>
-<part name="GND22" library="supply1" deviceset="GND" device=""/>
+<part name="U$3" library="crystal" deviceset="ASE" device=""/>
+<part name="GND74" library="supply1" deviceset="GND" device=""/>
+<part name="R11" library="rcl" deviceset="R-EU_" device="R0603"/>
 </parts>
 <sheets>
@@
 <instance part="GND26" gate="1" x="147.32" y="132.08"/>
 <instance part="R14" gate="G$1" x="17.78" y="289.56" rot="R180"/>
-<instance part="R15" gate="G$1" x="162.56" y="104.14"/>
+<instance part="R15" gate="G$1" x="129.54" y="292.1"/>
 <instance part="C29" gate="G$1" x="-35.56" y="190.5"/>
 <instance part="C30" gate="G$1" x="-134.62" y="190.5"/>
@@
 <instance part="U$4" gate="G$1" x="86.36" y="276.86"/>
 <instance part="GND9" gate="1" x="45.72" y="223.52"/>
-<instance part="C16" gate="G$1" x="-33.02" y="149.86"/>
-<instance part="C32" gate="G$1" x="-40.64" y="149.86"/>
-<instance part="GND17" gate="1" x="-33.02" y="132.08"/>
-<instance part="GND35" gate="1" x="-40.64" y="132.08"/>
-<instance part="Y1" gate="G$1" x="-33.02" y="160.02" rot="R90"/>
-<instance part="GND22" gate="1" x="-25.4" y="132.08"/>
+<instance part="U$3" gate="G$1" x="-93.98" y="152.4"/>
+<instance part="GND74" gate="1" x="-109.22" y="139.7"/>
+<instance part="R11" gate="G$1" x="-220.98" y="30.48" rot="R90"/>
 </instances>
 <busses>
@@
 </segment>
 <segment>
-<pinref part="C16" gate="G$1" pin="2"/>
-<pinref part="GND17" gate="1" pin="GND"/>
-<wire x1="-33.02" y1="134.62" x2="-33.02" y2="144.78" width="0.1524" layer="91"/>
-</segment>
-<segment>
-<pinref part="C32" gate="G$1" pin="2"/>
-<pinref part="GND35" gate="1" pin="GND"/>
-<wire x1="-40.64" y1="134.62" x2="-40.64" y2="144.78" width="0.1524" layer="91"/>
-</segment>
-<segment>
-<pinref part="Y1" gate="G$1" pin="3"/>
-<pinref part="GND22" gate="1" pin="GND"/>
-<wire x1="-27.94" y1="160.02" x2="-25.4" y2="160.02" width="0.1524" layer="91"/>
-<wire x1="-25.4" y1="160.02" x2="-25.4" y2="134.62" width="0.1524" layer="91"/>
+<pinref part="U$3" gate="G$1" pin="GND"/>
+<pinref part="GND74" gate="1" pin="GND"/>
+<wire x1="-106.68" y1="147.32" x2="-109.22" y2="147.32" width="0.1524" layer="91"/>
+<wire x1="-109.22" y1="147.32" x2="-109.22" y2="142.24" width="0.1524" layer="91"/>
 </segment>
 </net>
@@
 <segment>
 <pinref part="R15" gate="G$1" pin="2"/>
-<wire x1="167.64" y1="104.14" x2="170.18" y2="104.14" width="0.1524" layer="91"/>
-<label x="170.18" y="104.14" size="1.4224" layer="95" xref="yes"/>
+<wire x1="134.62" y1="292.1" x2="137.16" y2="292.1" width="0.1524" layer="91"/>
+<label x="137.16" y="292.1" size="1.4224" layer="95" xref="yes"/>
 </segment>
 <segment>
 <pinref part="U$4" gate="G$1" pin="VCC@1"/>
 <wire x1="86.36" y1="233.68" x2="86.36" y2="226.06" width="0.1524" layer="91"/>
+</segment>
+<segment>
+<pinref part="U$3" gate="G$1" pin="VDD"/>
+<wire x1="-106.68" y1="157.48" x2="-109.22" y2="157.48" width="0.1524" layer="91"/>
+<wire x1="-109.22" y1="157.48" x2="-109.22" y2="165.1" width="0.1524" layer="91"/>
+<label x="-109.22" y="165.1" size="1.4224" layer="95" rot="R90" xref="yes"/>
+</segment>
+<segment>
+<pinref part="R11" gate="G$1" pin="2"/>
+<wire x1="-220.98" y1="35.56" x2="-220.98" y2="38.1" width="0.1524" layer="91"/>
 </segment>
 </net>
@@
 <label x="-223.52" y="5.08" size="1.4224" layer="95" rot="R180" xref="yes"/>
 </segment>
+<segment>
+<pinref part="U$4" gate="G$1" pin="!IOE"/>
+<wire x1="106.68" y1="317.5" x2="106.68" y2="325.12" width="0.1524" layer="91"/>
+<label x="106.68" y="325.12" size="1.4224" layer="95" rot="R90" xref="yes"/>
+</segment>
 </net>
 <net name="!RD" class="0">
@@
 <pinref part="JP11" gate="A" pin="18"/>
 <wire x1="449.58" y1="152.4" x2="462.28" y2="152.4" width="0.1524" layer="91"/>
-</segment>
-<segment>
-<pinref part="IC4" gate="A" pin="G1"/>
-<wire x1="-218.44" y1="10.16" x2="-223.52" y2="10.16" width="0.1524" layer="91"/>
-<label x="-223.52" y="10.16" size="1.4224" layer="95" rot="R180" xref="yes"/>
 </segment>
 </net>
@@
 <net name="N$25" class="0">
 <segment>
-<wire x1="137.16" y1="104.14" x2="157.48" y2="104.14" width="0.1524" layer="91"/>
+<wire x1="121.92" y1="292.1" x2="124.46" y2="292.1" width="0.1524" layer="91"/>
 <pinref part="R15" gate="G$1" pin="1"/>
+<pinref part="U$4" gate="G$1" pin="!DREQ1"/>
 </segment>
 </net>
@@
 <label x="83.82" y="325.12" size="1.4224" layer="95" rot="R90" xref="yes"/>
 </segment>
-<segment>
-<wire x1="-20.32" y1="165.1" x2="-33.02" y2="165.1" width="0.1524" layer="91"/>
-<wire x1="-33.02" y1="165.1" x2="-33.02" y2="162.56" width="0.1524" layer="91"/>
-<pinref part="C32" gate="G$1" pin="1"/>
-<wire x1="-33.02" y1="165.1" x2="-40.64" y2="165.1" width="0.1524" layer="91"/>
-<wire x1="-40.64" y1="165.1" x2="-40.64" y2="152.4" width="0.1524" layer="91"/>
-<junction x="-33.02" y="165.1"/>
-<pinref part="Y1" gate="G$1" pin="2"/>
-<wire x1="-20.32" y1="165.1" x2="-12.7" y2="165.1" width="0.1524" layer="91"/>
-<label x="-12.7" y="165.1" size="1.4224" layer="95" xref="yes"/>
-</segment>
 </net>
 <net name="EXTAL" class="0">
@@
 </segment>
 <segment>
-<wire x1="-12.7" y1="154.94" x2="-33.02" y2="154.94" width="0.1524" layer="91"/>
-<wire x1="-33.02" y1="154.94" x2="-33.02" y2="157.48" width="0.1524" layer="91"/>
-<pinref part="C16" gate="G$1" pin="1"/>
-<wire x1="-33.02" y1="154.94" x2="-33.02" y2="152.4" width="0.1524" layer="91"/>
-<junction x="-33.02" y="154.94"/>
-<pinref part="Y1" gate="G$1" pin="1"/>
-<label x="-12.7" y="154.94" size="1.4224" layer="95" xref="yes"/>
-</segment>
-</net>
+<pinref part="U$3" gate="G$1" pin="OUT"/>
+<wire x1="-81.28" y1="152.4" x2="-73.66" y2="152.4" width="0.1524" layer="91"/>
+<label x="-73.66" y="152.4" size="1.4224" layer="95" rot="MR180" xref="yes"/>
+</segment>
+</net>
+<net name="N$26" class="0">
+<segment>
+<pinref part="IC4" gate="A" pin="G1"/>
+<pinref part="R11" gate="G$1" pin="1"/>
+<wire x1="-218.44" y1="10.16" x2="-220.98" y2="10.16" width="0.1524" layer="91"/>
+<wire x1="-220.98" y1="10.16" x2="-220.98" y2="25.4" width="0.1524" layer="91"/>
+</segment>
+</net>

Commit message: Local port added
Parts:
- added IC6: 74HCT273DW, 74xx-eu:74HCT273DW
- added IC8: 74LVC1G04DBV, 74xx-little-us:74LVC1G04DBV
- C27: device rcl:C-EUC0402 -> rcl:C-EUC0603
Connections:
- removed net CS7_NO_USE: IC4A.Y7
- new net LOCAL_PORT_CS: IC4A.Y7, IC8A.I
- new net N$44: IC6A.CLK, IC8A.O
- net !RST: now also IC6A.CLR
- net 5V: now also IC6P.VCC, IC8P.VCC
- net D4: now also IC6A.D4
- net D5: now also IC6A.D3
- net D6: now also IC6A.D2
- net D7: now also IC6A.D1
- net GND: now also IC6A.D5, IC6A.D6, IC6A.D7, IC6A.D8, IC6P.GND, IC8P.GND
- net RTS2: now also IC6A.Q1
Changed lines of the file:
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@@
 <part name="C24" library="rcl" deviceset="C-EU" device="C0603"/>
 <part name="C26" library="rcl" deviceset="C-EU" device="C0402"/>
-<part name="C27" library="rcl" deviceset="C-EU" device="C0402"/>
+<part name="C27" library="rcl" deviceset="C-EU" device="C0603"/>
 <part name="GND26" library="supply1" deviceset="GND" device=""/>
 <part name="R14" library="rcl" deviceset="R-EU_" device="0204/5"/>
@@
 <part name="GND74" library="supply1" deviceset="GND" device=""/>
 <part name="R11" library="rcl" deviceset="R-EU_" device="R0603"/>
+<part name="IC6" library="74xx-eu" deviceset="74*273" device="DW" technology="HCT" value="74HCT273DW"/>
+<part name="GND17" library="supply1" deviceset="GND" device=""/>
+<part name="IC8" library="74xx-little-us" deviceset="74*1G04" device="DBV" technology="LVC"/>
 </parts>
 <sheets>
@@
 <instance part="GND74" gate="1" x="-109.22" y="139.7"/>
 <instance part="R11" gate="G$1" x="-220.98" y="30.48" rot="R90"/>
+<instance part="IC6" gate="A" x="220.98" y="281.94"/>
+<instance part="GND17" gate="1" x="205.74" y="261.62"/>
+<instance part="IC6" gate="P" x="15.24" y="190.5"/>
+<instance part="IC8" gate="A" x="170.18" y="271.78"/>
+<instance part="IC8" gate="P" x="25.4" y="190.5"/>
 </instances>
 <busses>
@@
 <wire x1="5.08" y1="180.34" x2="5.08" y2="182.88" width="0.1524" layer="91"/>
 <junction x="-5.08" y="180.34"/>
+<pinref part="IC6" gate="P" pin="GND"/>
+<wire x1="5.08" y1="180.34" x2="15.24" y2="180.34" width="0.1524" layer="91"/>
+<wire x1="15.24" y1="180.34" x2="15.24" y2="182.88" width="0.1524" layer="91"/>
+<junction x="5.08" y="180.34"/>
+<pinref part="IC8" gate="P" pin="GND"/>
+<wire x1="15.24" y1="180.34" x2="25.4" y2="180.34" width="0.1524" layer="91"/>
+<wire x1="25.4" y1="180.34" x2="25.4" y2="182.88" width="0.1524" layer="91"/>
+<junction x="15.24" y="180.34"/>
 </segment>
 <segment>
@@
 <wire x1="-109.22" y1="147.32" x2="-109.22" y2="142.24" width="0.1524" layer="91"/>
 </segment>
+<segment>
+<pinref part="IC6" gate="A" pin="D5"/>
+<pinref part="GND17" gate="1" pin="GND"/>
+<wire x1="208.28" y1="284.48" x2="205.74" y2="284.48" width="0.1524" layer="91"/>
+<wire x1="205.74" y1="284.48" x2="205.74" y2="281.94" width="0.1524" layer="91"/>
+<pinref part="IC6" gate="A" pin="D6"/>
+<wire x1="205.74" y1="281.94" x2="205.74" y2="279.4" width="0.1524" layer="91"/>
+<wire x1="205.74" y1="279.4" x2="205.74" y2="276.86" width="0.1524" layer="91"/>
+<wire x1="205.74" y1="276.86" x2="205.74" y2="264.16" width="0.1524" layer="91"/>
+<wire x1="208.28" y1="281.94" x2="205.74" y2="281.94" width="0.1524" layer="91"/>
+<junction x="205.74" y="281.94"/>
+<pinref part="IC6" gate="A" pin="D7"/>
+<wire x1="208.28" y1="279.4" x2="205.74" y2="279.4" width="0.1524" layer="91"/>
+<junction x="205.74" y="279.4"/>
+<pinref part="IC6" gate="A" pin="D8"/>
+<wire x1="208.28" y1="276.86" x2="205.74" y2="276.86" width="0.1524" layer="91"/>
+<junction x="205.74" y="276.86"/>
+</segment>
 </net>
 <net name="5V" class="0">
@@
 <wire x1="5.08" y1="200.66" x2="5.08" y2="198.12" width="0.1524" layer="91"/>
 <junction x="-5.08" y="200.66"/>
+<pinref part="IC6" gate="P" pin="VCC"/>
+<wire x1="5.08" y1="200.66" x2="15.24" y2="200.66" width="0.1524" layer="91"/>
+<wire x1="15.24" y1="200.66" x2="15.24" y2="198.12" width="0.1524" layer="91"/>
+<junction x="5.08" y="200.66"/>
+<pinref part="IC8" gate="P" pin="VCC"/>
+<wire x1="15.24" y1="200.66" x2="25.4" y2="200.66" width="0.1524" layer="91"/>
+<wire x1="25.4" y1="200.66" x2="25.4" y2="198.12" width="0.1524" layer="91"/>
+<junction x="15.24" y="200.66"/>
 </segment>
 <segment>
@@
 <label x="152.4" y="109.22" size="1.4224" layer="95" xref="yes"/>
 </segment>
+<segment>
+<pinref part="IC6" gate="A" pin="Q1"/>
+<wire x1="233.68" y1="294.64" x2="241.3" y2="294.64" width="0.1524" layer="91"/>
+</segment>
 </net>
 <net name="RXD2" class="0">
@@
 <label x="104.14" y="226.06" size="1.4224" layer="95" rot="R270" xref="yes"/>
 </segment>
+<segment>
+<wire x1="208.28" y1="287.02" x2="200.66" y2="287.02" width="0.1524" layer="91"/>
+<label x="200.66" y="287.02" size="1.4224" layer="95" rot="R180" xref="yes"/>
+<pinref part="IC6" gate="A" pin="D4"/>
+</segment>
 </net>
 <net name="D5" class="0">
@@
 <label x="106.68" y="226.06" size="1.4224" layer="95" rot="R270" xref="yes"/>
 </segment>
+<segment>
+<wire x1="208.28" y1="289.56" x2="200.66" y2="289.56" width="0.1524" layer="91"/>
+<label x="200.66" y="289.56" size="1.4224" layer="95" rot="R180" xref="yes"/>
+<pinref part="IC6" gate="A" pin="D3"/>
+</segment>
 </net>
 <net name="D6" class="0">
@@
 <label x="132.08" y="246.38" size="1.4224" layer="95" xref="yes"/>
 </segment>
+<segment>
+<pinref part="IC6" gate="A" pin="D2"/>
+<wire x1="208.28" y1="292.1" x2="200.66" y2="292.1" width="0.1524" layer="91"/>
+<label x="200.66" y="292.1" size="1.4224" layer="95" rot="R180" xref="yes"/>
+</segment>
 </net>
 <net name="D7" class="0">
@@
 <wire x1="121.92" y1="254" x2="132.08" y2="254" width="0.1524" layer="91"/>
 <label x="132.08" y="254" size="1.4224" layer="95" xref="yes"/>
+</segment>
+<segment>
+<pinref part="IC6" gate="A" pin="D1"/>
+<wire x1="208.28" y1="294.64" x2="200.66" y2="294.64" width="0.1524" layer="91"/>
+<label x="200.66" y="294.64" size="1.4224" layer="95" rot="R180" xref="yes"/>
 </segment>
 </net>
@@
 <wire x1="68.58" y1="317.5" x2="68.58" y2="325.12" width="0.1524" layer="91"/>
 <label x="68.58" y="325.12" size="1.4224" layer="95" rot="R90" xref="yes"/>
+</segment>
+<segment>
+<pinref part="IC6" gate="A" pin="CLR"/>
+<wire x1="208.28" y1="269.24" x2="200.66" y2="269.24" width="0.1524" layer="91"/>
+<label x="200.66" y="269.24" size="1.4224" layer="95" rot="R180" xref="yes"/>
 </segment>
 </net>
@@
 </segment>
 </net>
-<net name="CS7_NO_USE" class="0">
-<segment>
-<pinref part="IC4" gate="A" pin="Y7"/>
-<wire x1="-190.5" y1="5.08" x2="-185.42" y2="5.08" width="0.1524" layer="91"/>
-<label x="-185.42" y="5.08" size="1.4224" layer="95" xref="yes"/>
-</segment>
-</net>
 <net name="XTAL" class="0">
 <segment>
@@
 </segment>
 </net>
+<net name="N$44" class="0">
+<segment>
+<pinref part="IC6" gate="A" pin="CLK"/>
+<pinref part="IC8" gate="A" pin="O"/>
+<wire x1="208.28" y1="271.78" x2="180.34" y2="271.78" width="0.1524" layer="91"/>
+</segment>
+</net>
+<net name="LOCAL_PORT_CS" class="0">
+<segment>
+<pinref part="IC8" gate="A" pin="I"/>
+<wire x1="160.02" y1="271.78" x2="154.94" y2="271.78" width="0.1524" layer="91"/>
+</segment>
+<segment>
+<pinref part="IC4" gate="A" pin="Y7"/>
+<wire x1="-190.5" y1="5.08" x2="-185.42" y2="5.08" width="0.1524" layer="91"/>
+<label x="-185.42" y="5.08" size="1.4224" layer="95" xref="yes"/>
+</segment>
+</net>
