File: hardware/cpu_board/untitled.sch (EAGLE design)
At the start: 73 parts, among them IC1 MAX232ECWE, IC2 MAX232ECWE, IC3 AM29F040J, IC4 74HCT138D, IC5 LM2596S, IC6 74HCT273DW, IC8 74LVC1G04DBV, J2 POWER_JACKSLT, U1 AS6C4008-55SIN

Commit message: E signal routed to edge connector
Connections:
- new net E: JP2.7, U$4.E
Changed lines of the file:
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@@
+</segment>
+</net>
+<net name="E" class="0">
+<segment>
+<pinref part="U$4" gate="G$1" pin="E"/>
+<wire x1="101.6" y1="317.5" x2="101.6" y2="325.12" width="0.1524" layer="91"/>
+</segment>
+<segment>
+<pinref part="JP2" gate="A" pin="7"/>
+<wire x1="457.2" y1="60.96" x2="447.04" y2="60.96" width="0.1524" layer="91"/>
 </segment>
 </net>

Commit message: Memory address decoder (work in progress)
Parts:
- added IC7: 74HCT139D, 74xx-eu:74HCT139D
- added R16: (no value), rcl:R-EU_R0603
Connections:
- new net !MEMEN: IC7B.G, U$4.!ME
- new net N$45: IC7B.B, R16.2
- new net ROMEN: IC6A.Q3, IC7B.A
- net 5V: now also IC7P.VCC
- net A15: now also R16.1
- net GND: now also IC7A.A, IC7A.B, IC7A.G, IC7P.GND
Changed lines of the file:
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@@
 <part name="GND17" library="supply1" deviceset="GND" device=""/>
 <part name="IC8" library="74xx-little-us" deviceset="74*1G04" device="DBV" technology="LVC"/>
+<part name="IC7" library="74xx-eu" deviceset="74*139" device="D" technology="HCT"/>
+<part name="GND22" library="supply1" deviceset="GND" device=""/>
+<part name="R16" library="rcl" deviceset="R-EU_" device="R0603"/>
 </parts>
 <sheets>
@@
 <instance part="IC8" gate="A" x="170.18" y="271.78"/>
 <instance part="IC8" gate="P" x="25.4" y="190.5"/>
+<instance part="IC7" gate="A" x="-205.74" y="-30.48"/>
+<instance part="IC7" gate="B" x="-205.74" y="-60.96"/>
+<instance part="IC7" gate="P" x="35.56" y="190.5"/>
+<instance part="GND22" gate="1" x="-220.98" y="-40.64"/>
+<instance part="R16" gate="G$1" x="-243.84" y="-60.96"/>
 </instances>
 <busses>
@@
 <wire x1="25.4" y1="180.34" x2="25.4" y2="182.88" width="0.1524" layer="91"/>
 <junction x="15.24" y="180.34"/>
+<pinref part="IC7" gate="P" pin="GND"/>
+<wire x1="25.4" y1="180.34" x2="35.56" y2="180.34" width="0.1524" layer="91"/>
+<wire x1="35.56" y1="180.34" x2="35.56" y2="182.88" width="0.1524" layer="91"/>
+<junction x="25.4" y="180.34"/>
 </segment>
 <segment>
@@
 <junction x="205.74" y="276.86"/>
 </segment>
+<segment>
+<pinref part="IC7" gate="A" pin="A"/>
+<pinref part="GND22" gate="1" pin="GND"/>
+<wire x1="-218.44" y1="-27.94" x2="-220.98" y2="-27.94" width="0.1524" layer="91"/>
+<wire x1="-220.98" y1="-27.94" x2="-220.98" y2="-30.48" width="0.1524" layer="91"/>
+<pinref part="IC7" gate="A" pin="G"/>
+<wire x1="-220.98" y1="-30.48" x2="-220.98" y2="-35.56" width="0.1524" layer="91"/>
+<wire x1="-220.98" y1="-35.56" x2="-220.98" y2="-38.1" width="0.1524" layer="91"/>
+<wire x1="-218.44" y1="-35.56" x2="-220.98" y2="-35.56" width="0.1524" layer="91"/>
+<junction x="-220.98" y="-35.56"/>
+<pinref part="IC7" gate="A" pin="B"/>
+<wire x1="-218.44" y1="-30.48" x2="-220.98" y2="-30.48" width="0.1524" layer="91"/>
+<junction x="-220.98" y="-30.48"/>
+</segment>
 </net>
 <net name="5V" class="0">
@@
 <wire x1="25.4" y1="200.66" x2="25.4" y2="198.12" width="0.1524" layer="91"/>
 <junction x="15.24" y="200.66"/>
+<pinref part="IC7" gate="P" pin="VCC"/>
+<wire x1="25.4" y1="200.66" x2="35.56" y2="200.66" width="0.1524" layer="91"/>
+<wire x1="35.56" y1="200.66" x2="35.56" y2="198.12" width="0.1524" layer="91"/>
+<junction x="25.4" y="200.66"/>
 </segment>
 <segment>
@@
 <label x="73.66" y="226.06" size="1.4224" layer="95" rot="R270" xref="yes"/>
 </segment>
+<segment>
+<pinref part="R16" gate="G$1" pin="1"/>
+<wire x1="-248.92" y1="-60.96" x2="-254" y2="-60.96" width="0.1524" layer="91"/>
+</segment>
 </net>
 <net name="TX" class="0">
@@
 </segment>
 </net>
+<net name="!MEMEN" class="0">
+<segment>
+<pinref part="U$4" gate="G$1" pin="!ME"/>
+<wire x1="104.14" y1="317.5" x2="104.14" y2="325.12" width="0.1524" layer="91"/>
+</segment>
+<segment>
+<pinref part="IC7" gate="B" pin="G"/>
+<wire x1="-218.44" y1="-66.04" x2="-223.52" y2="-66.04" width="0.1524" layer="91"/>
+<label x="-223.52" y="-66.04" size="1.4224" layer="95" rot="R180" xref="yes"/>
+</segment>
+</net>
+<net name="ROMEN" class="0">
+<segment>
+<pinref part="IC7" gate="B" pin="A"/>
+<wire x1="-218.44" y1="-58.42" x2="-223.52" y2="-58.42" width="0.1524" layer="91"/>
+<label x="-223.52" y="-58.42" size="1.4224" layer="95" rot="R180" xref="yes"/>
+</segment>
+<segment>
+<pinref part="IC6" gate="A" pin="Q3"/>
+<wire x1="233.68" y1="289.56" x2="241.3" y2="289.56" width="0.1524" layer="91"/>
+</segment>
+</net>
+<net name="N$45" class="0">
+<segment>
+<pinref part="IC7" gate="B" pin="B"/>
+<pinref part="R16" gate="G$1" pin="2"/>
+<wire x1="-218.44" y1="-60.96" x2="-238.76" y2="-60.96" width="0.1524" layer="91"/>
+</segment>
+</net>

Commit message: Minor changes
Parts:
- removed IC7: 74HCT139D, 74xx-eu:74HCT139D
Connections:
- removed net N$45: IC7B.B, R16.2
- removed net ROMEN: IC6A.Q3, IC7B.A
- new net ROMSHADOW: IC6A.Q3
- new net _A15: R16.2
- net !MEMEN: no longer IC7B.G
- net 5V: no longer IC7P.VCC
- net GND: no longer IC7A.A, IC7A.B, IC7A.G, IC7P.GND
Other:
- moved on the sheet: R16
Changed lines of the file:
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@@
 <part name="GND17" library="supply1" deviceset="GND" device=""/>
 <part name="IC8" library="74xx-little-us" deviceset="74*1G04" device="DBV" technology="LVC"/>
-<part name="IC7" library="74xx-eu" deviceset="74*139" device="D" technology="HCT"/>
-<part name="GND22" library="supply1" deviceset="GND" device=""/>
 <part name="R16" library="rcl" deviceset="R-EU_" device="R0603"/>
 </parts>
@@
 <instance part="IC8" gate="A" x="170.18" y="271.78"/>
 <instance part="IC8" gate="P" x="25.4" y="190.5"/>
-<instance part="IC7" gate="A" x="-205.74" y="-30.48"/>
-<instance part="IC7" gate="B" x="-205.74" y="-60.96"/>
-<instance part="IC7" gate="P" x="35.56" y="190.5"/>
-<instance part="GND22" gate="1" x="-220.98" y="-40.64"/>
-<instance part="R16" gate="G$1" x="-243.84" y="-60.96"/>
+<instance part="R16" gate="G$1" x="-220.98" y="-50.8"/>
 </instances>
 <busses>
@@
 <wire x1="25.4" y1="180.34" x2="25.4" y2="182.88" width="0.1524" layer="91"/>
 <junction x="15.24" y="180.34"/>
-<pinref part="IC7" gate="P" pin="GND"/>
-<wire x1="25.4" y1="180.34" x2="35.56" y2="180.34" width="0.1524" layer="91"/>
-<wire x1="35.56" y1="180.34" x2="35.56" y2="182.88" width="0.1524" layer="91"/>
-<junction x="25.4" y="180.34"/>
 </segment>
 <segment>
@@
 <junction x="205.74" y="276.86"/>
 </segment>
-<segment>
-<pinref part="IC7" gate="A" pin="A"/>
-<pinref part="GND22" gate="1" pin="GND"/>
-<wire x1="-218.44" y1="-27.94" x2="-220.98" y2="-27.94" width="0.1524" layer="91"/>
-<wire x1="-220.98" y1="-27.94" x2="-220.98" y2="-30.48" width="0.1524" layer="91"/>
-<pinref part="IC7" gate="A" pin="G"/>
-<wire x1="-220.98" y1="-30.48" x2="-220.98" y2="-35.56" width="0.1524" layer="91"/>
-<wire x1="-220.98" y1="-35.56" x2="-220.98" y2="-38.1" width="0.1524" layer="91"/>
-<wire x1="-218.44" y1="-35.56" x2="-220.98" y2="-35.56" width="0.1524" layer="91"/>
-<junction x="-220.98" y="-35.56"/>
-<pinref part="IC7" gate="A" pin="B"/>
-<wire x1="-218.44" y1="-30.48" x2="-220.98" y2="-30.48" width="0.1524" layer="91"/>
-<junction x="-220.98" y="-30.48"/>
-</segment>
 </net>
 <net name="5V" class="0">
@@
 <wire x1="25.4" y1="200.66" x2="25.4" y2="198.12" width="0.1524" layer="91"/>
 <junction x="15.24" y="200.66"/>
-<pinref part="IC7" gate="P" pin="VCC"/>
-<wire x1="25.4" y1="200.66" x2="35.56" y2="200.66" width="0.1524" layer="91"/>
-<wire x1="35.56" y1="200.66" x2="35.56" y2="198.12" width="0.1524" layer="91"/>
-<junction x="25.4" y="200.66"/>
 </segment>
 <segment>
@@
 <segment>
 <pinref part="R16" gate="G$1" pin="1"/>
-<wire x1="-248.92" y1="-60.96" x2="-254" y2="-60.96" width="0.1524" layer="91"/>
+<wire x1="-226.06" y1="-50.8" x2="-228.6" y2="-50.8" width="0.1524" layer="91"/>
 </segment>
 </net>
@@
 <wire x1="104.14" y1="317.5" x2="104.14" y2="325.12" width="0.1524" layer="91"/>
 </segment>
-<segment>
-<pinref part="IC7" gate="B" pin="G"/>
-<wire x1="-218.44" y1="-66.04" x2="-223.52" y2="-66.04" width="0.1524" layer="91"/>
-<label x="-223.52" y="-66.04" size="1.4224" layer="95" rot="R180" xref="yes"/>
-</segment>
-</net>
-<net name="ROMEN" class="0">
-<segment>
-<pinref part="IC7" gate="B" pin="A"/>
-<wire x1="-218.44" y1="-58.42" x2="-223.52" y2="-58.42" width="0.1524" layer="91"/>
-<label x="-223.52" y="-58.42" size="1.4224" layer="95" rot="R180" xref="yes"/>
-</segment>
+</net>
+<net name="ROMSHADOW" class="0">
 <segment>
 <pinref part="IC6" gate="A" pin="Q3"/>
@@
 </segment>
 </net>
-<net name="N$45" class="0">
-<segment>
-<pinref part="IC7" gate="B" pin="B"/>
+<net name="_A15" class="0">
+<segment>
 <pinref part="R16" gate="G$1" pin="2"/>
-<wire x1="-218.44" y1="-60.96" x2="-238.76" y2="-60.96" width="0.1524" layer="91"/>
-</segment>
-</net>
+<wire x1="-208.28" y1="-50.8" x2="-215.9" y2="-50.8" width="0.1524" layer="91"/>
+</segment>
+</net>

Commit message: Writing to 273 fixed
Parts:
- added IC7: 74LVC1G08DBV, 74xx-little-de:74LVC1G08DBV
- C26: device rcl:C-EUC0402 -> rcl:C-EUC0603
Connections:
- new net N$45: IC7A.I0, IC8A.O
- net !WR: now also IC7A.I1
- net 5V: now also IC7P.VCC
- net GND: now also IC7P.GND
- net N$44: now also IC7A.O; no longer IC8A.O
Other:
- moved on the sheet: IC6, IC8
Changed lines of the file:
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@@
 <part name="JP8" library="pinhead" deviceset="PINHD-1X2" device=""/>
 <part name="C24" library="rcl" deviceset="C-EU" device="C0603"/>
-<part name="C26" library="rcl" deviceset="C-EU" device="C0402"/>
+<part name="C26" library="rcl" deviceset="C-EU" device="C0603"/>
 <part name="C27" library="rcl" deviceset="C-EU" device="C0603"/>
 <part name="GND26" library="supply1" deviceset="GND" device=""/>
@@
 <part name="IC8" library="74xx-little-us" deviceset="74*1G04" device="DBV" technology="LVC"/>
 <part name="R16" library="rcl" deviceset="R-EU_" device="R0603"/>
+<part name="IC7" library="74xx-little-de" deviceset="74*1G08" device="DBV" technology="LVC"/>
 </parts>
 <sheets>
@@
 <instance part="GND74" gate="1" x="-109.22" y="139.7"/>
 <instance part="R11" gate="G$1" x="-220.98" y="30.48" rot="R90"/>
-<instance part="IC6" gate="A" x="220.98" y="281.94"/>
-<instance part="GND17" gate="1" x="205.74" y="261.62"/>
+<instance part="IC6" gate="A" x="264.16" y="281.94"/>
+<instance part="GND17" gate="1" x="248.92" y="261.62"/>
 <instance part="IC6" gate="P" x="15.24" y="190.5"/>
-<instance part="IC8" gate="A" x="170.18" y="271.78"/>
+<instance part="IC8" gate="A" x="182.88" y="274.32"/>
 <instance part="IC8" gate="P" x="25.4" y="190.5"/>
 <instance part="R16" gate="G$1" x="-220.98" y="-50.8"/>
+<instance part="IC7" gate="A" x="203.2" y="271.78"/>
+<instance part="IC7" gate="P" x="35.56" y="190.5"/>
 </instances>
 <busses>
@@
 <wire x1="25.4" y1="180.34" x2="25.4" y2="182.88" width="0.1524" layer="91"/>
 <junction x="15.24" y="180.34"/>
+<pinref part="IC7" gate="P" pin="GND"/>
+<wire x1="25.4" y1="180.34" x2="35.56" y2="180.34" width="0.1524" layer="91"/>
+<wire x1="35.56" y1="180.34" x2="35.56" y2="182.88" width="0.1524" layer="91"/>
+<junction x="25.4" y="180.34"/>
 </segment>
 <segment>
@@
 <pinref part="IC6" gate="A" pin="D5"/>
 <pinref part="GND17" gate="1" pin="GND"/>
-<wire x1="208.28" y1="284.48" x2="205.74" y2="284.48" width="0.1524" layer="91"/>
-<wire x1="205.74" y1="284.48" x2="205.74" y2="281.94" width="0.1524" layer="91"/>
+<wire x1="251.46" y1="284.48" x2="248.92" y2="284.48" width="0.1524" layer="91"/>
+<wire x1="248.92" y1="284.48" x2="248.92" y2="281.94" width="0.1524" layer="91"/>
 <pinref part="IC6" gate="A" pin="D6"/>
-<wire x1="205.74" y1="281.94" x2="205.74" y2="279.4" width="0.1524" layer="91"/>
-<wire x1="205.74" y1="279.4" x2="205.74" y2="276.86" width="0.1524" layer="91"/>
-<wire x1="205.74" y1="276.86" x2="205.74" y2="264.16" width="0.1524" layer="91"/>
-<wire x1="208.28" y1="281.94" x2="205.74" y2="281.94" width="0.1524" layer="91"/>
-<junction x="205.74" y="281.94"/>
+<wire x1="248.92" y1="281.94" x2="248.92" y2="279.4" width="0.1524" layer="91"/>
+<wire x1="248.92" y1="279.4" x2="248.92" y2="276.86" width="0.1524" layer="91"/>
+<wire x1="248.92" y1="276.86" x2="248.92" y2="264.16" width="0.1524" layer="91"/>
+<wire x1="251.46" y1="281.94" x2="248.92" y2="281.94" width="0.1524" layer="91"/>
+<junction x="248.92" y="281.94"/>
 <pinref part="IC6" gate="A" pin="D7"/>
-<wire x1="208.28" y1="279.4" x2="205.74" y2="279.4" width="0.1524" layer="91"/>
-<junction x="205.74" y="279.4"/>
+<wire x1="251.46" y1="279.4" x2="248.92" y2="279.4" width="0.1524" layer="91"/>
+<junction x="248.92" y="279.4"/>
 <pinref part="IC6" gate="A" pin="D8"/>
-<wire x1="208.28" y1="276.86" x2="205.74" y2="276.86" width="0.1524" layer="91"/>
-<junction x="205.74" y="276.86"/>
+<wire x1="251.46" y1="276.86" x2="248.92" y2="276.86" width="0.1524" layer="91"/>
+<junction x="248.92" y="276.86"/>
 </segment>
 </net>
@@
 <wire x1="25.4" y1="200.66" x2="25.4" y2="198.12" width="0.1524" layer="91"/>
 <junction x="15.24" y="200.66"/>
+<pinref part="IC7" gate="P" pin="VCC"/>
+<wire x1="25.4" y1="200.66" x2="35.56" y2="200.66" width="0.1524" layer="91"/>
+<wire x1="35.56" y1="200.66" x2="35.56" y2="198.12" width="0.1524" layer="91"/>
+<junction x="25.4" y="200.66"/>
 </segment>
 <segment>
@@
 <segment>
 <pinref part="IC6" gate="A" pin="Q1"/>
-<wire x1="233.68" y1="294.64" x2="241.3" y2="294.64" width="0.1524" layer="91"/>
+<wire x1="276.86" y1="294.64" x2="284.48" y2="294.64" width="0.1524" layer="91"/>
 </segment>
 </net>
@@
 </segment>
 <segment>
-<wire x1="208.28" y1="287.02" x2="200.66" y2="287.02" width="0.1524" layer="91"/>
-<label x="200.66" y="287.02" size="1.4224" layer="95" rot="R180" xref="yes"/>
+<wire x1="251.46" y1="287.02" x2="243.84" y2="287.02" width="0.1524" layer="91"/>
+<label x="243.84" y="287.02" size="1.4224" layer="95" rot="R180" xref="yes"/>
 <pinref part="IC6" gate="A" pin="D4"/>
 </segment>
@@
 </segment>
 <segment>
-<wire x1="208.28" y1="289.56" x2="200.66" y2="289.56" width="0.1524" layer="91"/>
-<label x="200.66" y="289.56" size="1.4224" layer="95" rot="R180" xref="yes"/>
+<wire x1="251.46" y1="289.56" x2="243.84" y2="289.56" width="0.1524" layer="91"/>
+<label x="243.84" y="289.56" size="1.4224" layer="95" rot="R180" xref="yes"/>
 <pinref part="IC6" gate="A" pin="D3"/>
 </segment>
@@
 <segment>
 <pinref part="IC6" gate="A" pin="D2"/>
-<wire x1="208.28" y1="292.1" x2="200.66" y2="292.1" width="0.1524" layer="91"/>
-<label x="200.66" y="292.1" size="1.4224" layer="95" rot="R180" xref="yes"/>
+<wire x1="251.46" y1="292.1" x2="243.84" y2="292.1" width="0.1524" layer="91"/>
+<label x="243.84" y="292.1" size="1.4224" layer="95" rot="R180" xref="yes"/>
 </segment>
 </net>
@@
 <segment>
 <pinref part="IC6" gate="A" pin="D1"/>
-<wire x1="208.28" y1="294.64" x2="200.66" y2="294.64" width="0.1524" layer="91"/>
-<label x="200.66" y="294.64" size="1.4224" layer="95" rot="R180" xref="yes"/>
+<wire x1="251.46" y1="294.64" x2="243.84" y2="294.64" width="0.1524" layer="91"/>
+<label x="243.84" y="294.64" size="1.4224" layer="95" rot="R180" xref="yes"/>
 </segment>
 </net>
@@
 <wire x1="96.52" y1="317.5" x2="96.52" y2="325.12" width="0.1524" layer="91"/>
 <label x="96.52" y="325.12" size="1.4224" layer="95" rot="R90" xref="yes"/>
+</segment>
+<segment>
+<pinref part="IC7" gate="A" pin="I1"/>
+<wire x1="198.12" y1="269.24" x2="193.04" y2="269.24" width="0.1524" layer="91"/>
 </segment>
 </net>
@@
 <segment>
 <pinref part="IC6" gate="A" pin="CLR"/>
-<wire x1="208.28" y1="269.24" x2="200.66" y2="269.24" width="0.1524" layer="91"/>
-<label x="200.66" y="269.24" size="1.4224" layer="95" rot="R180" xref="yes"/>
+<wire x1="251.46" y1="269.24" x2="243.84" y2="269.24" width="0.1524" layer="91"/>
+<label x="243.84" y="269.24" size="1.4224" layer="95" rot="R180" xref="yes"/>
 </segment>
 </net>
@@
 </segment>
 </net>
-<net name="N$44" class="0">
-<segment>
-<pinref part="IC6" gate="A" pin="CLK"/>
-<pinref part="IC8" gate="A" pin="O"/>
-<wire x1="208.28" y1="271.78" x2="180.34" y2="271.78" width="0.1524" layer="91"/>
-</segment>
-</net>
 <net name="LOCAL_PORT_CS" class="0">
 <segment>
 <pinref part="IC8" gate="A" pin="I"/>
-<wire x1="160.02" y1="271.78" x2="154.94" y2="271.78" width="0.1524" layer="91"/>
+<wire x1="172.72" y1="274.32" x2="157.48" y2="274.32" width="0.1524" layer="91"/>
 </segment>
 <segment>
@@
 <segment>
 <pinref part="IC6" gate="A" pin="Q3"/>
-<wire x1="233.68" y1="289.56" x2="241.3" y2="289.56" width="0.1524" layer="91"/>
+<wire x1="276.86" y1="289.56" x2="284.48" y2="289.56" width="0.1524" layer="91"/>
 </segment>
 </net>
@@
 </segment>
 </net>
+<net name="N$44" class="0">
+<segment>
+<pinref part="IC6" gate="A" pin="CLK"/>
+<pinref part="IC7" gate="A" pin="O"/>
+<wire x1="210.82" y1="271.78" x2="251.46" y2="271.78" width="0.1524" layer="91"/>
+</segment>
+</net>
+<net name="N$45" class="0">
+<segment>
+<pinref part="IC7" gate="A" pin="I0"/>
+<pinref part="IC8" gate="A" pin="O"/>
+<wire x1="193.04" y1="274.32" x2="198.12" y2="274.32" width="0.1524" layer="91"/>
+</segment>
+</net>
