File: hardware/cpu_board/untitled.sch (EAGLE design)
At the start: 82 parts, among them IC1 MAX232ECWE, IC2 MAX232ECWE, IC3 AM29F040J, IC4 74HCT138D, IC5 LM2596S, IC6 74HCT273DW, IC7 74LVC1G08DBV, IC8 74LVC1G04DBV, IC9 74HCT138D, J2 POWER_JACKSLT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

Commit message: PCB bug fix
Parts:
- removed C26: (no value), rcl:C-EUC0603
- removed IC8: 74LVC1G04DBV, 74xx-little-us:74LVC1G04DBV
- IC7: value 74LVC1G08DBV -> 74AHC1G02DBV; device 74xx-little-de:74LVC1G08DBV -> 74xx-little-de:74AHC1G02DBV
Connections:
- removed net N$45: IC7A.I0, IC8A.O
- net 5V: no longer C26.1, IC8P.VCC
- net GND: no longer C26.2, IC8P.GND
- net LOCAL_PORT_CS: now also IC7A.I0; no longer IC8A.I
Other:
- moved on the sheet: C27, C29, C3, IC7P, IC9P
Changed lines of the file:
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@@
 <part name="JP8" library="pinhead" deviceset="PINHD-1X2" device=""/>
 <part name="C24" library="rcl" deviceset="C-EU" device="C0603"/>
-<part name="C26" library="rcl" deviceset="C-EU" device="C0603"/>
 <part name="C27" library="rcl" deviceset="C-EU" device="C0603"/>
 <part name="GND26" library="supply1" deviceset="GND" device=""/>
@@
 <part name="IC6" library="74xx-eu" deviceset="74*273" device="DW" technology="HCT" value="74HCT273DW"/>
 <part name="GND17" library="supply1" deviceset="GND" device=""/>
-<part name="IC8" library="74xx-little-us" deviceset="74*1G04" device="DBV" technology="LVC"/>
 <part name="R16" library="rcl" deviceset="R-EU_" device="R0603"/>
-<part name="IC7" library="74xx-little-de" deviceset="74*1G08" device="DBV" technology="LVC"/>
+<part name="IC7" library="74xx-little-de" deviceset="74*1G02" device="DBV" technology="AHC" value="74AHC1G02DBV"/>
 <part name="R17" library="rcl" deviceset="R-EU_" device="R0603"/>
 <part name="LED1" library="led" deviceset="LED" device="CHIP-LED0603"/>
@@
 <instance part="JP8" gate="G$1" x="-248.92" y="284.48" rot="R90"/>
 <instance part="C24" gate="G$1" x="-66.04" y="190.5"/>
-<instance part="C26" gate="G$1" x="-58.42" y="190.5"/>
-<instance part="C27" gate="G$1" x="-50.8" y="190.5"/>
+<instance part="C27" gate="G$1" x="-58.42" y="190.5"/>
 <instance part="GND26" gate="1" x="147.32" y="132.08"/>
 <instance part="R14" gate="G$1" x="17.78" y="289.56" rot="R180"/>
 <instance part="R15" gate="G$1" x="129.54" y="292.1"/>
-<instance part="C29" gate="G$1" x="-43.18" y="190.5"/>
+<instance part="C29" gate="G$1" x="-50.8" y="190.5"/>
 <instance part="C30" gate="G$1" x="-127" y="190.5"/>
 <instance part="C31" gate="G$1" x="-134.62" y="190.5"/>
@@
 <instance part="GND17" gate="1" x="248.92" y="261.62"/>
 <instance part="IC6" gate="P" x="15.24" y="190.5"/>
-<instance part="IC8" gate="A" x="182.88" y="274.32"/>
-<instance part="IC8" gate="P" x="25.4" y="190.5"/>
 <instance part="R16" gate="G$1" x="-210.82" y="-38.1"/>
 <instance part="IC7" gate="A" x="203.2" y="271.78"/>
-<instance part="IC7" gate="P" x="35.56" y="190.5"/>
+<instance part="IC7" gate="P" x="25.4" y="190.5"/>
 <instance part="R17" gate="G$1" x="284.48" y="287.02" rot="R180"/>
 <instance part="LED1" gate="G$1" x="294.64" y="287.02" rot="R90"/>
@@
 <instance part="GND23" gate="1" x="-203.2" y="-55.88"/>
 <instance part="R18" gate="G$1" x="-200.66" y="-25.4" rot="R90"/>
-<instance part="IC9" gate="P" x="45.72" y="190.5"/>
+<instance part="IC9" gate="P" x="35.56" y="190.5"/>
 <instance part="D2" gate="G$1" x="-162.56" y="-38.1" rot="R180"/>
 <instance part="D3" gate="G$1" x="-162.56" y="-43.18" rot="R180"/>
 <instance part="D4" gate="G$1" x="-162.56" y="-48.26" rot="R180"/>
 <instance part="R19" gate="G$1" x="-152.4" y="-22.86" rot="R90"/>
-<instance part="C3" gate="G$1" x="-35.56" y="190.5"/>
+<instance part="C3" gate="G$1" x="-43.18" y="190.5"/>
 </instances>
 <busses>
@@
 <wire x1="15.24" y1="180.34" x2="15.24" y2="182.88" width="0.1524" layer="91"/>
 <junction x="5.08" y="180.34"/>
-<pinref part="IC8" gate="P" pin="GND"/>
+<junction x="15.24" y="180.34"/>
+<pinref part="IC7" gate="P" pin="GND"/>
 <wire x1="15.24" y1="180.34" x2="25.4" y2="180.34" width="0.1524" layer="91"/>
 <wire x1="25.4" y1="180.34" x2="25.4" y2="182.88" width="0.1524" layer="91"/>
-<junction x="15.24" y="180.34"/>
-<pinref part="IC7" gate="P" pin="GND"/>
+<pinref part="IC9" gate="P" pin="GND"/>
 <wire x1="25.4" y1="180.34" x2="35.56" y2="180.34" width="0.1524" layer="91"/>
 <wire x1="35.56" y1="180.34" x2="35.56" y2="182.88" width="0.1524" layer="91"/>
 <junction x="25.4" y="180.34"/>
-<pinref part="IC9" gate="P" pin="GND"/>
-<wire x1="35.56" y1="180.34" x2="45.72" y2="180.34" width="0.1524" layer="91"/>
-<wire x1="45.72" y1="180.34" x2="45.72" y2="182.88" width="0.1524" layer="91"/>
-<junction x="35.56" y="180.34"/>
 </segment>
 <segment>
@@
 <wire x1="-66.04" y1="182.88" x2="-66.04" y2="185.42" width="0.1524" layer="91"/>
 <junction x="-73.66" y="182.88"/>
-<pinref part="C26" gate="G$1" pin="2"/>
+<junction x="-66.04" y="182.88"/>
+<pinref part="C27" gate="G$1" pin="2"/>
 <wire x1="-66.04" y1="182.88" x2="-58.42" y2="182.88" width="0.1524" layer="91"/>
 <wire x1="-58.42" y1="182.88" x2="-58.42" y2="185.42" width="0.1524" layer="91"/>
-<junction x="-66.04" y="182.88"/>
-<pinref part="C27" gate="G$1" pin="2"/>
+<pinref part="C29" gate="G$1" pin="2"/>
 <wire x1="-58.42" y1="182.88" x2="-50.8" y2="182.88" width="0.1524" layer="91"/>
 <wire x1="-50.8" y1="182.88" x2="-50.8" y2="185.42" width="0.1524" layer="91"/>
 <junction x="-58.42" y="182.88"/>
-<pinref part="C29" gate="G$1" pin="2"/>
-<wire x1="-50.8" y1="182.88" x2="-43.18" y2="182.88" width="0.1524" layer="91"/>
-<wire x1="-43.18" y1="182.88" x2="-43.18" y2="185.42" width="0.1524" layer="91"/>
-<junction x="-50.8" y="182.88"/>
 <pinref part="C30" gate="G$1" pin="-"/>
 <wire x1="-119.38" y1="182.88" x2="-127" y2="182.88" width="0.1524" layer="91"/>
@@
 <junction x="-127" y="182.88"/>
 <pinref part="C3" gate="G$1" pin="2"/>
-<wire x1="-43.18" y1="182.88" x2="-35.56" y2="182.88" width="0.1524" layer="91"/>
-<wire x1="-35.56" y1="182.88" x2="-35.56" y2="185.42" width="0.1524" layer="91"/>
-<junction x="-43.18" y="182.88"/>
+<wire x1="-50.8" y1="182.88" x2="-43.18" y2="182.88" width="0.1524" layer="91"/>
+<wire x1="-43.18" y1="182.88" x2="-43.18" y2="185.42" width="0.1524" layer="91"/>
+<junction x="-50.8" y="182.88"/>
 </segment>
 <segment>
@@
 <wire x1="15.24" y1="200.66" x2="15.24" y2="198.12" width="0.1524" layer="91"/>
 <junction x="5.08" y="200.66"/>
-<pinref part="IC8" gate="P" pin="VCC"/>
+<junction x="15.24" y="200.66"/>
+<pinref part="IC7" gate="P" pin="VCC"/>
 <wire x1="15.24" y1="200.66" x2="25.4" y2="200.66" width="0.1524" layer="91"/>
 <wire x1="25.4" y1="200.66" x2="25.4" y2="198.12" width="0.1524" layer="91"/>
-<junction x="15.24" y="200.66"/>
-<pinref part="IC7" gate="P" pin="VCC"/>
+<pinref part="IC9" gate="P" pin="VCC"/>
 <wire x1="25.4" y1="200.66" x2="35.56" y2="200.66" width="0.1524" layer="91"/>
 <wire x1="35.56" y1="200.66" x2="35.56" y2="198.12" width="0.1524" layer="91"/>
 <junction x="25.4" y="200.66"/>
-<pinref part="IC9" gate="P" pin="VCC"/>
-<wire x1="35.56" y1="200.66" x2="45.72" y2="200.66" width="0.1524" layer="91"/>
-<wire x1="45.72" y1="200.66" x2="45.72" y2="198.12" width="0.1524" layer="91"/>
-<junction x="35.56" y="200.66"/>
 </segment>
 <segment>
@@
 <wire x1="-66.04" y1="195.58" x2="-66.04" y2="193.04" width="0.1524" layer="91"/>
 <junction x="-73.66" y="195.58"/>
-<pinref part="C26" gate="G$1" pin="1"/>
+<junction x="-66.04" y="195.58"/>
+<pinref part="C27" gate="G$1" pin="1"/>
 <wire x1="-66.04" y1="195.58" x2="-58.42" y2="195.58" width="0.1524" layer="91"/>
 <wire x1="-58.42" y1="195.58" x2="-58.42" y2="193.04" width="0.1524" layer="91"/>
-<junction x="-66.04" y="195.58"/>
-<pinref part="C27" gate="G$1" pin="1"/>
+<pinref part="C29" gate="G$1" pin="1"/>
 <wire x1="-58.42" y1="195.58" x2="-50.8" y2="195.58" width="0.1524" layer="91"/>
 <wire x1="-50.8" y1="195.58" x2="-50.8" y2="193.04" width="0.1524" layer="91"/>
 <junction x="-58.42" y="195.58"/>
-<pinref part="C29" gate="G$1" pin="1"/>
-<wire x1="-50.8" y1="195.58" x2="-43.18" y2="195.58" width="0.1524" layer="91"/>
-<wire x1="-43.18" y1="195.58" x2="-43.18" y2="193.04" width="0.1524" layer="91"/>
-<junction x="-50.8" y="195.58"/>
 <pinref part="C30" gate="G$1" pin="+"/>
 <wire x1="-119.38" y1="195.58" x2="-127" y2="195.58" width="0.1524" layer="91"/>
@@
 <junction x="-127" y="195.58"/>
 <pinref part="C3" gate="G$1" pin="1"/>
-<wire x1="-43.18" y1="195.58" x2="-35.56" y2="195.58" width="0.1524" layer="91"/>
-<wire x1="-35.56" y1="195.58" x2="-35.56" y2="193.04" width="0.1524" layer="91"/>
-<junction x="-43.18" y="195.58"/>
+<wire x1="-50.8" y1="195.58" x2="-43.18" y2="195.58" width="0.1524" layer="91"/>
+<wire x1="-43.18" y1="195.58" x2="-43.18" y2="193.04" width="0.1524" layer="91"/>
+<junction x="-50.8" y="195.58"/>
 </segment>
 <segment>
@@
 <pinref part="IC7" gate="A" pin="I1"/>
 <wire x1="198.12" y1="269.24" x2="193.04" y2="269.24" width="0.1524" layer="91"/>
+<label x="193.04" y="269.24" size="1.4224" layer="95" rot="R180" xref="yes"/>
 </segment>
 </net>
@@
 <net name="LOCAL_PORT_CS" class="0">
 <segment>
-<pinref part="IC8" gate="A" pin="I"/>
-<wire x1="172.72" y1="274.32" x2="157.48" y2="274.32" width="0.1524" layer="91"/>
+<label x="193.04" y="274.32" size="1.4224" layer="95" rot="R180" xref="yes"/>
+<pinref part="IC7" gate="A" pin="I0"/>
+<wire x1="193.04" y1="274.32" x2="198.12" y2="274.32" width="0.1524" layer="91"/>
 </segment>
 <segment>
@@
 </segment>
 </net>
-<net name="N$45" class="0">
-<segment>
-<pinref part="IC7" gate="A" pin="I0"/>
-<pinref part="IC8" gate="A" pin="O"/>
-<wire x1="193.04" y1="274.32" x2="198.12" y2="274.32" width="0.1524" layer="91"/>
-</segment>
-</net>
